File: modem_rf.kicad_sch (KiCad schematic)
At the start: 64 parts, among them Q10 MMBT3904, Q11 MMBT3904, Q12 MMBT3904, Q13 MMBT3906, Q14 MMBT3904, Q3 AO3401A, Q9 MMBT3904, U1 EC200UCNAA-N05-SGNSA, U8 TXB0104PWR, X1 NANO-SIM, X2 MFF2-eSIM-pads

Commit message: F-21 RETRACTED (my misread); antennas selected; 8 of 8 floorplan checks pass
F-21 was wrong and the error was mine. I read the pdftotext -layout dump, where
0R and 100 pF share a row and NM NM sit below, and took the 100 pF for a shunt.
Rendering page 69 at 200 dpi shows it has VERTICAL plates in the signal line: it
is a SERIES DC BLOCK, and the 47 nH injects VDD on the ANTENNA side of it. The
module pin is DC-isolated by construction; there was never a conflict.
Corroborated by Antenna Design Guide V3.3 5.1 note 5, which also asks for
>= 56 nH - so L4 is 68 nH, not figure 31's 47 nH. Table 40 does not list
ANT_GNSS at all, so there is no published DC rating for pin 47, which is the
real reason the block is mandatory.

Schematic corrected: C84 100 pF is in SERIES and ALWAYS FITTED (depopulating it
opens the antenna; 1.0 ohm at 1575 MHz). Only L4/R90/C83 are DNP. Chain verified
in the netlist: U1.47 -> R72 -> C84 -> AF2.3, bias injected at ANT_GNSS_F.
C84 anchored inline in the RF corridor and check 1 extended to validate every
inline element. checkpins caught a real short while doing this - the first
bias-T placement merged GNSS_BIAS into USIM_VDD.

Parts: C1546 100pF C0G (always fitted), C3221844 Murata LQW15AN68NG80D 68 nH
WIREWOUND SRF 2.5 GHz (every multilayer 0402 at this value has SRF ~1.1 GHz and
is capacitive at 1575 MHz), C25077 10R, C60474 0.1uF.

Antennas: LTE C496569 Bat Wireless BW4GFNX39-15B1, 700-2700 MHz continuous,
120 mm IPEX-1 pigtail, 5536 stock. Runner-up C22467619 rejected - it omits B40,
which Jio uses heavily in India.

GNSS C784386 - but this is a DEVIATION NEEDING A DECISION: no passive 25x25
patch with a U.FL pigtail exists in LCSC stock, so the recommendation is ACTIVE
(LNA 21.5 dB, 1.8-3.6 V, 4.3 mA). That makes the bias-T MANDATORY rather than
DNP for the internal build. Passive alternative C784398 has solder pins and no
cable, needing a hand-added pigtail and a 60-70 mm lid ground plane.

Quectel's < 17 dB LNA limit is a recommendation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
Parts:
- C83: value 100nF DNP -> 100nF
- C84: value 100pF DNP -> 100pF C0G; LCSC TBD-F21 -> C1546; now fitted
- L4: value 47nH DNP -> 68nH; LCSC TBD-F21 -> C3221844
- R90: value 10R DNP -> 10R; LCSC TBD-F21 -> C25077
Connections:
- net ANT_GNSS_C: no longer AF2.3 (SIG), L4.1
- net GND: no longer C84.2
- new net ANT_GNSS_F: AF2.3 (SIG), C84.2, L4.1
Other:
- note added: "GNSS: C84 100pF SERIES DC BLOCK IS ALWAYS FITTED (Quectel fig 31). L4/R90/C83 are the bias-T, DNP - fit only for an active antenna. 68nH per Antenna Design Guide >=56nH; must be WIREWOUND (multilayer 0402 SRF is ~1.1GHz, useless)."
- note removed: "GNSS bias-T (DNP): Quectel V1.2 fig 31 - 47nH series, 100pF shunt, 10R+100nF on the 3V3 feed. Fit ONLY for an active external antenna; see F-21 on the DC block."
- moved on the sheet: C83, L4, R90
Changed lines of the file:
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@@
 	(wire
 		(pts
-			(xy 302.26 176.53) (xy 302.26 172.72)
+			(xy 304.8 199.39) (xy 304.8 195.58)
 		)
 		(stroke
@@
 	)
 	(label "ANT_GNSS_C"
-		(at 302.26 172.72 90)
+		(at 304.8 195.58 90)
 		(effects
 			(font
@@
 	(wire
 		(pts
-			(xy 302.26 184.15) (xy 302.26 187.96)
+			(xy 304.8 207.01) (xy 304.8 210.82)
 		)
 		(stroke
@@
 		)
 	)
-	(label "GNSS_BIAS"
-		(at 302.26 187.96 270)
+	(label "ANT_GNSS_F"
+		(at 304.8 210.82 270)
 		(effects
 			(font
@@
 	(wire
 		(pts
-			(xy 312.42 166.37) (xy 312.42 162.56)
+			(xy 345.44 199.39) (xy 345.44 195.58)
 		)
 		(stroke
@@
 		)
 	)
-	(label "3V3"
-		(at 312.42 162.56 90)
+	(label "ANT_GNSS_F"
+		(at 345.44 195.58 90)
 		(effects
 			(font
@@
 	(wire
 		(pts
-			(xy 312.42 173.99) (xy 312.42 177.8)
+			(xy 345.44 207.01) (xy 345.44 210.82)
 		)
 		(stroke
@@
 	)
 	(label "GNSS_BIAS"
-		(at 312.42 177.8 270)
+		(at 345.44 210.82 270)
 		(effects
 			(font
@@
 	(wire
 		(pts
-			(xy 302.26 161.29) (xy 302.26 157.48)
+			(xy 365.76 186.69) (xy 365.76 182.88)
 		)
 		(stroke
@@
 		)
 	)
-	(label "GNSS_BIAS"
-		(at 302.26 157.48 90)
+	(label "3V3"
+		(at 365.76 182.88 90)
 		(effects
 			(font
@@
 	(wire
 		(pts
-			(xy 302.26 168.91) (xy 302.26 171.45)
+			(xy 365.76 194.31) (xy 365.76 198.12)
 		)
 		(stroke
@@
 		)
 	)
+	(label "GNSS_BIAS"
+		(at 365.76 198.12 270)
+		(effects
+			(font
+				(size 1.27 1.27)
+			)
+			(justify right bottom)
+		)
+	)
 	(wire
 		(pts
-			(xy 289.56 176.53) (xy 289.56 172.72)
+			(xy 350.52 181.61) (xy 350.52 177.8)
 		)
 		(stroke
@@
 		)
 	)
-	(label "ANT_GNSS_C"
-		(at 289.56 172.72 90)
+	(label "GNSS_BIAS"
+		(at 350.52 177.8 90)
 		(effects
 			(font
@@
 	(wire
 		(pts
-			(xy 289.56 184.15) (xy 289.56 186.69)
+			(xy 350.52 189.23) (xy 350.52 191.77)
 		)
 		(stroke
@@
 		)
 	)
-	(text "GNSS bias-T (DNP): Quectel V1.2 fig 31 - 47nH series, 100pF shunt, 10R+100nF on the 3V3 feed. Fit ONLY for an active external antenna; see F-21 on the DC block."
+	(text "GNSS: C84 100pF SERIES DC BLOCK IS ALWAYS FITTED (Quectel fig 31). L4/R90/C83 are the bias-T, DNP - fit only for an active antenna. 68nH per Antenna Design Guide >=56nH; must be WIREWOUND (multilayer 0402 SRF is ~1.1GHz, useless)."
 		(exclude_from_sim no)
-		(at 279.4 157.48 0)
+		(at 330.2 175.26 0)
 		(effects
 			(font
@@
 		)
 	)
-	(label "ANT_GNSS_C"
+	(label "ANT_GNSS_F"
 		(at 323.85 194.31 0)
 		(effects
@@
 	)
 	(symbol
-		(lib_id "Device:L")
-		(at 302.26 180.34 0)
+		(lib_id "Device:C")
+		(at 304.8 203.2 0)
 		(unit 1)
 		(exclude_from_sim no)
 		(in_bom yes)
 		(on_board yes)
-		(dnp yes)
+		(dnp no)
 		(fields_autoplaced yes)
-		(property "Reference" "L4"
-			(at 302.26 177.8 0)
+		(property "Reference" "C84"
+			(at 304.8 200.66 0)
 			(effects
 				(font
@@
 			)
 		)
-		(property "Value" "47nH DNP"
-			(at 302.26 175.26 0)
+		(property "Value" "100pF C0G"
+			(at 304.8 198.12 0)
 			(effects
 				(font
@@
 			)
 		)
-		(property "Footprint" "Inductor_SMD:L_0402_1005Metric"
-			(at 302.26 180.34 0)
+		(property "Footprint" "Capacitor_SMD:C_0402_1005Metric"
+			(at 304.8 203.2 0)
 			(hide yes)
 			(effects
@@
 		)
 		(property "Datasheet" "~"
-			(at 302.26 180.34 0)
+			(at 304.8 203.2 0)
 			(hide yes)
 			(effects
@@
 			)
 		)
-		(property "LCSC" "TBD-F21"
-			(at 302.26 180.34 0)
+		(property "LCSC" "C1546"
+			(at 304.8 203.2 0)
 			(hide yes)
 			(effects
@@
 			(project "telematics-tracker"
 				(path "/784bc421-9fc7-43cb-bfc3-562714cb3f68/70fac1b9-7bfc-5985-a8dc-ae866bd73e38"
-					(reference "L4")
+					(reference "C84")
 					(unit 1)
 				)
@@
 	)
 	(symbol
-		(lib_id "Device:R")
-		(at 312.42 170.18 0)
+		(lib_id "Device:L")
+		(at 345.44 203.2 0)
 		(unit 1)
 		(exclude_from_sim no)
@@
 		(dnp yes)
 		(fields_autoplaced yes)
-		(property "Reference" "R90"
-			(at 312.42 167.64 0)
+		(property "Reference" "L4"
+			(at 345.44 200.66 0)
 			(effects
 				(font
@@
 			)
 		)
-		(property "Value" "10R DNP"
-			(at 312.42 165.1 0)
+		(property "Value" "68nH"
+			(at 345.44 198.12 0)
 			(effects
 				(font
@@
 			)
 		)
-		(property "Footprint" "Resistor_SMD:R_0402_1005Metric"
-			(at 312.42 170.18 0)
+		(property "Footprint" "Inductor_SMD:L_0402_1005Metric"
+			(at 345.44 203.2 0)
 			(hide yes)
 			(effects
@@
 		)
 		(property "Datasheet" "~"
-			(at 312.42 170.18 0)
+			(at 345.44 203.2 0)
 			(hide yes)
 			(effects
@@
 			)
 		)
-		(property "LCSC" "TBD-F21"
-			(at 312.42 170.18 0)
+		(property "LCSC" "C3221844"
+			(at 345.44 203.2 0)
 			(hide yes)
 			(effects
@@
 			(project "telematics-tracker"
 				(path "/784bc421-9fc7-43cb-bfc3-562714cb3f68/70fac1b9-7bfc-5985-a8dc-ae866bd73e38"
-					(reference "R90")
+					(reference "L4")
 					(unit 1)
 				)
@@
 	)
 	(symbol
-		(lib_id "Device:C")
-		(at 302.26 165.1 0)
+		(lib_id "Device:R")
+		(at 365.76 190.5 0)
 		(unit 1)
 		(exclude_from_sim no)
@@
 		(dnp yes)
 		(fields_autoplaced yes)
-		(property "Reference" "C83"
-			(at 302.26 162.56 0)
+		(property "Reference" "R90"
+			(at 365.76 187.96 0)
 			(effects
 				(font
@@
 			)
 		)
-		(property "Value" "100nF DNP"
-			(at 302.26 160.02 0)
+		(property "Value" "10R"
+			(at 365.76 185.42 0)
 			(effects
 				(font
@@
 			)
 		)
-		(property "Footprint" "Capacitor_SMD:C_0402_1005Metric"
-			(at 302.26 165.1 0)
+		(property "Footprint" "Resistor_SMD:R_0402_1005Metric"
+			(at 365.76 190.5 0)
 			(hide yes)
 			(effects
@@
 		)
 		(property "Datasheet" "~"
-			(at 302.26 165.1 0)
+			(at 365.76 190.5 0)
 			(hide yes)
 			(effects
@@
 			)
 		)
-		(property "LCSC" "C14663"
-			(at 302.26 165.1 0)
+		(property "LCSC" "C25077"
+			(at 365.76 190.5 0)
 			(hide yes)
 			(effects
@@
 			(project "telematics-tracker"
 				(path "/784bc421-9fc7-43cb-bfc3-562714cb3f68/70fac1b9-7bfc-5985-a8dc-ae866bd73e38"
-					(reference "C83")
-					(unit 1)
-				)
-			)
-		)
-	)
-	(symbol
-		(lib_id "power:GND")
-		(at 302.26 171.45 0)
-		(unit 1)
-		(exclude_from_sim no)
-		(in_bom yes)
-		(on_board yes)
-		(dnp no)
-		(fields_autoplaced yes)
-		(property "Reference" "#PWR147"
-			(at 302.26 163.83 0)
-			(effects
-				(font
-					(size 1.27 1.27)
-				)
-			)
-		)
-		(property "Value" "GND"
-			(at 302.26 171.45 0)
-			(hide yes)
-			(effects
-				(font
-					(size 1.27 1.27)
-				)
-			)
-		)
-		(pin "1"
-		)
-		(instances
-			(project "telematics-tracker"
-				(path "/784bc421-9fc7-43cb-bfc3-562714cb3f68/70fac1b9-7bfc-5985-a8dc-ae866bd73e38"
-					(reference "#PWR147")
+					(reference "R90")
 					(unit 1)
 				)
@@
 	(symbol
 		(lib_id "Device:C")
-		(at 289.56 180.34 0)
+		(at 350.52 185.42 0)
 		(unit 1)
 		(exclude_from_sim no)
@@
 		(dnp yes)
 		(fields_autoplaced yes)
-		(property "Reference" "C84"
-			(at 289.56 177.8 0)
+		(property "Reference" "C83"
+			(at 350.52 182.88 0)
 			(effects
 				(font
@@
 			)
 		)
-		(property "Value" "100pF DNP"
-			(at 289.56 175.26 0)
+		(property "Value" "100nF"
+			(at 350.52 180.34 0)
 			(effects
 				(font
@@
 		)
 		(property "Footprint" "Capacitor_SMD:C_0402_1005Metric"
-			(at 289.56 180.34 0)
+			(at 350.52 185.42 0)
 			(hide yes)
 			(effects
@@
 		)
 		(property "Datasheet" "~"
-			(at 289.56 180.34 0)
+			(at 350.52 185.42 0)
 			(hide yes)
 			(effects
@@
 			)
 		)
-		(property "LCSC" "TBD-F21"
-			(at 289.56 180.34 0)
+		(property "LCSC" "C14663"
+			(at 350.52 185.42 0)
 			(hide yes)
 			(effects
@@
 			(project "telematics-tracker"
 				(path "/784bc421-9fc7-43cb-bfc3-562714cb3f68/70fac1b9-7bfc-5985-a8dc-ae866bd73e38"
-					(reference "C84")
+					(reference "C83")
 					(unit 1)
 				)
@@
 	(symbol
 		(lib_id "power:GND")
-		(at 289.56 186.69 0)
+		(at 350.52 191.77 0)
 		(unit 1)
 		(exclude_from_sim no)
@@
 		(dnp no)
 		(fields_autoplaced yes)
-		(property "Reference" "#PWR148"
-			(at 289.56 179.07 0)
+		(property "Reference" "#PWR147"
+			(at 350.52 184.15 0)
 			(effects
 				(font
@@
 		)
 		(property "Value" "GND"
-			(at 289.56 186.69 0)
+			(at 350.52 191.77 0)
 			(hide yes)
 			(effects
@@
 			(project "telematics-tracker"
 				(path "/784bc421-9fc7-43cb-bfc3-562714cb3f68/70fac1b9-7bfc-5985-a8dc-ae866bd73e38"
-					(reference "#PWR148")
+					(reference "#PWR147")
 					(unit 1)
 				)
@@
 		(dnp no)
 		(fields_autoplaced yes)
-		(property "Reference" "#PWR149"
+		(property "Reference" "#PWR148"
 			(at 300.99 184.15 0)
 			(effects
@@
 			(project "telematics-tracker"
 				(path "/784bc421-9fc7-43cb-bfc3-562714cb3f68/70fac1b9-7bfc-5985-a8dc-ae866bd73e38"
-					(reference "#PWR149")
+					(reference "#PWR148")
 					(unit 1)
 				)
@@
 		(dnp no)
 		(fields_autoplaced yes)
-		(property "Reference" "#PWR150"
+		(property "Reference" "#PWR149"
 			(at 300.99 186.69 0)
 			(effects
@@
 			(project "telematics-tracker"
 				(path "/784bc421-9fc7-43cb-bfc3-562714cb3f68/70fac1b9-7bfc-5985-a8dc-ae866bd73e38"
-					(reference "#PWR150")
+					(reference "#PWR149")
 					(unit 1)
 				)

Commit message: Pre-routing: R90 short protection, bias-T on all builds, F-23 antenna temp
Bias-T POPULATED on all builds - the selected GNSS antenna C784386 is active
(LNA 21.5 dB, 1.8-3.6 V), so L4/R90/C83 are no longer DNP. C84 100pF series DC
block was already always-fitted.

R90 antenna-short current limit = 68R 1210 (F-22). The vendor publishes only a
TYPICAL 4.3 mA and no maximum, so this is designed to a conservative multiple:
  normal, 3V3 at -5%: V_ant = 2.84 V at 1x typical, still 1.95 V at 4x typical
                      (needs >= 1.80 V) - tolerates 4.3x the typical current
  fault, 3V3 at +5%:  50.1 mA into a shorted coax, vs a 500 mA LDO already
                      carrying ~150 mA, and L4 rated 320 mA
  P_R90 in fault:     0.171 W, 68% of a 50%-derated 1210
Deliberately more conservative than the ~150 mA brief: 22R would hit 143 mA but
needs a 2512 and burns 0.448 W CONTINUOUSLY inside a sealed IP65 box at 70 C,
from a fault that does not clear itself. C85 10nF added at the injection node
because 68R (vs Quectel's 10R) raises supply-noise coupling into the LNA.

F-23 NEW - the antennas are the weakest thermal link. Both are -45 to +85 C for
OPERATING AND STORAGE (identical ranges, verified verbatim in both datasheets).
That gives 15 C margin at the +70 C operating limit but ZERO margin at the 85 C
survival limit, with no excursion or derating data published by either vendor.
They are lid-mounted, i.e. in the hottest part of the enclosure. Bench soak at
85 C required before release; decision open on whether to accept, narrow the
survival spec, or treat antennas as serviceable.

Antenna retention must be MECHANICAL - heat stake, clamp, rib or captive pocket,
never adhesive alone (Quectel Antenna Design Guide V3.3 3.1 note 3: adhesive
weakens at high ambient). Added to the installation sheet AND as a housing
selection criterion in handoff 6.3 and 7 - the enclosure must provide the
retention feature, so a plain smooth-lidded box will not do.

Also noted: both datashe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
Parts:
- added C85: 10nF, Capacitor_SMD:C_0402_1005Metric, symbol Device:C
- C83, L4: now fitted
- R90: value 10R -> 68R; footprint Resistor_SMD:R_0402_1005Metric -> Resistor_SMD:R_1210_3225Metric; LCSC C25077 -> TBD-F22; now fitted
Connections:
- net GND: now also C85.2
- net GNSS_BIAS: now also C85.1
Other:
- note added: "GNSS bias-T POPULATED ON ALL BUILDS - antenna C784386 is ACTIVE (LNA 21.5dB, 1.8-3.6V). C84 100pF is the SERIES DC BLOCK (Quectel fig 31), always fitted. L4 68nH per Antenna Design Guide >=56nH, must be WIREWOUND. R90 is the antenna-short current limit - see design-log."
- note removed: "GNSS: C84 100pF SERIES DC BLOCK IS ALWAYS FITTED (Quectel fig 31). L4/R90/C83 are the bias-T, DNP - fit only for an active antenna. 68nH per Antenna Design Guide >=56nH; must be WIREWOUND (multilayer 0402 SRF is ~1.1GHz, useless)."
Changed lines of the file:
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@@
 		)
 	)
-	(text "GNSS: C84 100pF SERIES DC BLOCK IS ALWAYS FITTED (Quectel fig 31). L4/R90/C83 are the bias-T, DNP - fit only for an active antenna. 68nH per Antenna Design Guide >=56nH; must be WIREWOUND (multilayer 0402 SRF is ~1.1GHz, useless)."
+	(wire
+		(pts
+			(xy 358.14 181.61) (xy 358.14 177.8)
+		)
+		(stroke
+			(width 0)
+			(type default)
+		)
+	)
+	(label "GNSS_BIAS"
+		(at 358.14 177.8 90)
+		(effects
+			(font
+				(size 1.27 1.27)
+			)
+			(justify left bottom)
+		)
+	)
+	(wire
+		(pts
+			(xy 358.14 189.23) (xy 358.14 191.77)
+		)
+		(stroke
+			(width 0)
+			(type default)
+		)
+	)
+	(text "GNSS bias-T POPULATED ON ALL BUILDS - antenna C784386 is ACTIVE (LNA 21.5dB, 1.8-3.6V). C84 100pF is the SERIES DC BLOCK (Quectel fig 31), always fitted. L4 68nH per Antenna Design Guide >=56nH, must be WIREWOUND. R90 is the antenna-short current limit - see design-log."
 		(exclude_from_sim no)
 		(at 330.2 175.26 0)
@@
 		(in_bom yes)
 		(on_board yes)
-		(dnp yes)
+		(dnp no)
 		(fields_autoplaced yes)
 		(property "Reference" "L4"
@@
 		(in_bom yes)
 		(on_board yes)
-		(dnp yes)
+		(dnp no)
 		(fields_autoplaced yes)
 		(property "Reference" "R90"
@@
 			)
 		)
-		(property "Value" "10R"
+		(property "Value" "68R"
 			(at 365.76 185.42 0)
 			(effects
@@
 			)
 		)
-		(property "Footprint" "Resistor_SMD:R_0402_1005Metric"
+		(property "Footprint" "Resistor_SMD:R_1210_3225Metric"
 			(at 365.76 190.5 0)
 			(hide yes)
@@
 			)
 		)
-		(property "LCSC" "C25077"
+		(property "LCSC" "TBD-F22"
 			(at 365.76 190.5 0)
 			(hide yes)
@@
 		(in_bom yes)
 		(on_board yes)
-		(dnp yes)
+		(dnp no)
 		(fields_autoplaced yes)
 		(property "Reference" "C83"
@@
 	)
 	(symbol
+		(lib_id "Device:C")
+		(at 358.14 185.42 0)
+		(unit 1)
+		(exclude_from_sim no)
+		(in_bom yes)
+		(on_board yes)
+		(dnp no)
+		(fields_autoplaced yes)
+		(property "Reference" "C85"
+			(at 358.14 182.88 0)
+			(effects
+				(font
+					(size 1.27 1.27)
+				)
+			)
+		)
+		(property "Value" "10nF"
+			(at 358.14 180.34 0)
+			(effects
+				(font
+					(size 1.27 1.27)
+				)
+			)
+		)
+		(property "Footprint" "Capacitor_SMD:C_0402_1005Metric"
+			(at 358.14 185.42 0)
+			(hide yes)
+			(effects
+				(font
+					(size 1.27 1.27)
+				)
+			)
+		)
+		(property "Datasheet" "~"
+			(at 358.14 185.42 0)
+			(hide yes)
+			(effects
+				(font
+					(size 1.27 1.27)
+				)
+			)
+		)
+		(property "LCSC" "TBD-F22"
+			(at 358.14 185.42 0)
+			(hide yes)
+			(effects
+				(font
+					(size 1.27 1.27)
+				)
+			)
+		)
+		(pin "1"
+		)
+		(pin "2"
+		)
+		(instances
+			(project "telematics-tracker"
+				(path "/784bc421-9fc7-43cb-bfc3-562714cb3f68/70fac1b9-7bfc-5985-a8dc-ae866bd73e38"
+					(reference "C85")
+					(unit 1)
+				)
+			)
+		)
+	)
+	(symbol
+		(lib_id "power:GND")
+		(at 358.14 191.77 0)
+		(unit 1)
+		(exclude_from_sim no)
+		(in_bom yes)
+		(on_board yes)
+		(dnp no)
+		(fields_autoplaced yes)
+		(property "Reference" "#PWR148"
+			(at 358.14 184.15 0)
+			(effects
+				(font
+					(size 1.27 1.27)
+				)
+			)
+		)
+		(property "Value" "GND"
+			(at 358.14 191.77 0)
+			(hide yes)
+			(effects
+				(font
+					(size 1.27 1.27)
+				)
+			)
+		)
+		(pin "1"
+		)
+		(instances
+			(project "telematics-tracker"
+				(path "/784bc421-9fc7-43cb-bfc3-562714cb3f68/70fac1b9-7bfc-5985-a8dc-ae866bd73e38"
+					(reference "#PWR148")
+					(unit 1)
+				)
+			)
+		)
+	)
+	(symbol
 		(lib_id "jlc:XY-IPEX1")
 		(at 312.42 193.04 0)
@@
 		(dnp no)
 		(fields_autoplaced yes)
-		(property "Reference" "#PWR148"
+		(property "Reference" "#PWR149"
 			(at 300.99 184.15 0)
 			(effects
@@
 			(project "telematics-tracker"
 				(path "/784bc421-9fc7-43cb-bfc3-562714cb3f68/70fac1b9-7bfc-5985-a8dc-ae866bd73e38"
-					(reference "#PWR148")
+					(reference "#PWR149")
 					(unit 1)
 				)
@@
 		(dnp no)
 		(fields_autoplaced yes)
-		(property "Reference" "#PWR149"
+		(property "Reference" "#PWR150"
 			(at 300.99 186.69 0)
 			(effects
@@
 			(project "telematics-tracker"
 				(path "/784bc421-9fc7-43cb-bfc3-562714cb3f68/70fac1b9-7bfc-5985-a8dc-ae866bd73e38"
-					(reference "#PWR149")
+					(reference "#PWR150")
 					(unit 1)
 				)

Commit message: Step 1-3: fix rule floors, classify SW_BUCK as HV, shrink, fix HV router
Step 1 - rule mismatch fixed and verified:
  netclasses.py gains BOARD_RULES + _assert_floors(). Every class now meets
  track >= 0.20 mm and via annulus >= 0.10 mm. min_clearance had been silently
  reset to 0.0 by a KiCad round trip; restored to 0.15 and now asserted after
  the round trip so it cannot regress unnoticed. Exported DSN verified to carry
  the values (kicad_default 200, GND 500, MODEM_BULK 2000, RF 400, HV 500/600).

Step 2 - HV hand-routing, and three real defects it uncovered:

  1. /power/SW_BUCK was in the Default netclass. It is the buck switching node:
     it swings from GND to VIN every cycle, so it is a 100 V net with fast
     edges, and it was running at 0.20 mm track / 0.15 mm clearance. U5_VB
     (bootstrap) rides on it and was equally misclassified. Both moved to HV.
     Found because the maze router treated SW_BUCK as LV and threw a 1.50 mm
     halo around U5's own VIN pins, making /power/VIN_B unroutable at 0/4.

  2. HV_ZONE stopped at x = 20.0 and so EXCLUDED the buck primary side. U5 sits
     at x 35.4..42.3 with C73, C74 and D16 beside it, and VIN_B runs 22 mm from
     R80 to reach it. The highest-energy node on the board was outside the HV
     rule area - which also meant the U5 package exception approved under F-20
     was dead code, since it is conditioned on insideArea('HV_ZONE'). HV_ZONE
     is now L-shaped: left strip plus the buck primary.

  3. Three defects in pcbroute_hv.py itself, together responsible for 128 of
     the 129 clearance violations the first routed board had:
       - halos were sized for a 0.50 mm track (half 0.25) but the router also
         drops 0.80 mm vias, so cells legal for a track were illegal for a via
       - halo extents were quantised with round(), letting a cell centre sit up
         to RES/2 = 0.075 mm inside the forbidden region. That is exactly the
         size of the 0.545..0.594 mm shortfalls DRC reporte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
Parts:
- removed TP14: MODEM_STATUS, TestPoint:TestPoint_Pad_D1.5mm, symbol Connector:TestPoint
