File: modem_rf.kicad_sch (KiCad schematic)
At the start: 64 parts, among them Q10 MMBT3904, Q11 MMBT3904, Q12 MMBT3904, Q13 MMBT3906, Q14 MMBT3904, Q3 AO3401A, Q9 MMBT3904, U1 EC200UCNAA-N05-SGNSA, U8 TXB0104PWR, X1 NANO-SIM, X2 MFF2-eSIM-pads

Commit message: BOM verification (milestone 5): 28 wrong or unverified lines fixed against LCSC/JLCPCB data; F-5 and F-22 closed
Wrong values (C1/C2 22pF for 18pF, C3/C4, R56/R58 10k for 47k, R66-R68
100R for 33R), wrong packages (C12/C63, C83, R71/R72, Y1 5032 on a 3225
footprint), Y2 12.5pF crystal on 6.8pF caps (now a 7pF FC-135), red LED
number on the green and blue LEDs (R4/R6 330R for their Vf), a
non-existent C-number (2.2k), and nine TBD placeholders.

tools/bom_audit.py: value / voltage / package / LED colour / crystal load /
stock (JLCPCB and LCSC) per line -> docs/bom-audit.md, out/bom-mpn.csv
(manufacturer + MPN). Netlist connectivity unchanged, ERC 0, checkpins ok.

Co-Authored-By: Claude Opus 5.5 <noreply@anthropic.com>
Parts:
- C83: LCSC C14663 -> C1525
- C85: LCSC TBD-F22 -> C15195
- R56, R58: LCSC C17414 -> C17713
- R66, R67, R68: LCSC C17408 -> C17634
- R71, R72: LCSC C17477 -> C17168
- R90: LCSC TBD-F22 -> C137091
Changed lines of the file:
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@@
 			)
 		)
-		(property "LCSC" "C17414"
+		(property "LCSC" "C17713"
 			(at 38.1 165.1 0)
 			(hide yes)
@@
 			)
 		)
-		(property "LCSC" "C17414"
+		(property "LCSC" "C17713"
 			(at 73.66 165.1 0)
 			(hide yes)
@@
 			)
 		)
-		(property "LCSC" "C17408"
+		(property "LCSC" "C17634"
 			(at 294.64 76.2 0)
 			(hide yes)
@@
 			)
 		)
-		(property "LCSC" "C17408"
+		(property "LCSC" "C17634"
 			(at 307.34 76.2 0)
 			(hide yes)
@@
 			)
 		)
-		(property "LCSC" "C17408"
+		(property "LCSC" "C17634"
 			(at 320.04 76.2 0)
 			(hide yes)
@@
 			)
 		)
-		(property "LCSC" "C17477"
+		(property "LCSC" "C17168"
 			(at 241.3 203.2 0)
 			(hide yes)
@@
 			)
 		)
-		(property "LCSC" "C17477"
+		(property "LCSC" "C17168"
 			(at 292.1 203.2 0)
 			(hide yes)
@@
 			)
 		)
-		(property "LCSC" "TBD-F22"
+		(property "LCSC" "C137091"
 			(at 365.76 190.5 0)
 			(hide yes)
@@
 			)
 		)
-		(property "LCSC" "C14663"
+		(property "LCSC" "C1525"
 			(at 350.52 185.42 0)
 			(hide yes)
@@
 			)
 		)
-		(property "LCSC" "TBD-F22"
+		(property "LCSC" "C15195"
 			(at 358.14 185.42 0)
 			(hide yes)

Commit message: Pre-order verification review: 12 would-fail faults fixed, report added
Schematic (tools/sheets.py, sheets regenerated):
- D2 SMDJ100A: D_Zener symbol, cathode to VIN_P (was drawn forward with
  the bidirectional D_TVS symbol)
- D10/D11 BAV99 clamps: pin 1 (anode) GND, pin 2 (cathode) 3V3 (KiCad's
  hidden K/A/K pin names contradict the Nexperia pinout)
- D5/D6: BAV70 common-cathode replaces the mirrored BAV99 (opto LED was
  bypassed)
- U8 TXB0104 OE: 10k/100k = 1.64 V (47k/10k gave 0.32 V, UART disabled)
- R82 0.1R: EG11752 2 A peak limit (0R disabled it)
- D7/D8 flyback cathodes to VIN_P behind D1 (reverse-polarity path via
  the Q1/Q2 body diodes), VIN_P exported as a hierarchical net
- Q1/Q2 gate pulldown 100k (4.89 V; 10k gave 4.07 V), DI pull-up 220k,
  R91 51k USIM_DET pull-up, PESD5V0L5UY SIM ESD, X7R 1uF/4.7uF, 100k
  C149504, comments and notes corrected

Board (DRC-gated routes via tools/manual_routes.py + tools/board_fixes.py):
- D2/D10/D11 turned, NRST via moved, VIN trunk re-laid around D7/D8,
  VIN_P B.Cu run to D1, R91 on B.Cu, VBAT_BT 0.6 mm F.Cu to J2, SW_CHG
  0.4 mm, PMID 0.3/0.5 mm, DNP flags, C61<->C80 swap, 28 RF stitching
  vias, 9 vias under U5's pad; values updated
- manual_routes: delvia/padnet/rotate/value/move ops, ACCEPT_EQUAL

Checks: parity 0 mismatches (212 parts, 727 pad nets), ERC 0 errors,
pin checklist pass, DRC 0 errors / 0 unconnected, BOM audit 76/76 clean.

Docs: firmware-notes FW-6/8/13/14/17 + FW-18..22, BV-1/5/6/7; handoff and
installation sheet corrected (12 V floor, DI not isolated, values);
design-log entry; docs/verification-report.pdf (OK / NOT OK per item).

Co-Authored-By: Claude Fable 5.1 <noreply@anthropic.com>
Parts:
- added R91: 51k, Resistor_SMD:R_0603_1608Metric, symbol Device:R
- C42, C44: LCSC C15849 -> C106858
- D14: value SMF05C -> PESD5V0L5UY; LCSC C15879 -> C179747
- R50: LCSC C17407 -> C149504
- R62: value 10k -> 100k; LCSC C17414 -> C149504
- R63: value 47k -> 10k; LCSC C17713 -> C17414
Connections:
- net USIM_DET: now also R91.2
- net VDD_EXT_1V8: now also R91.1
Other:
- note added: "U8 TXB0104: A=1.8V (VDD_EXT), B=3V3. A1<->B1 carries MCU TX -> modem MAIN_RXD(68); A2<->B2 modem MAIN_TXD(67) -> MCU RX; A3 RI(62); A4 DTR(66). OE = 10k/100k from VDD_EXT (1.64 V)."
- note added: "USIM: 33R series on DATA/CLK/RST, 100nF on VDD, PESD5V0L5UY (19pF) at the holder, 51k USIM_DET pull-up to VDD_EXT. MFF2 eSIM pads (X2, DNP) parallel; VDD via 0R selects R69 (fitted, holder) / R70 (DNP, eSIM)."
- note added: "VBAT_MODEM: 4x47uF X7R (F-13) + 1uF + 100nF + SMF5.0A, place <=5mm from U1 VBAT pads (57-60)."
- note removed: "U8 TXB0104: A=1.8V (VDD_EXT), B=3V3. A1<->B1 carries MCU TX -> modem MAIN_RXD(68); A2<->B2 modem MAIN_TXD(67) -> MCU RX; A3 RI(62); A4 DTR(66). OE held low until VDD_EXT rises."
- note removed: "USIM: 33R series on DATA/CLK/RST, 100nF on VDD, SMF05C at the holder. MFF2 eSIM pads (X2, DNP) parallel; VDD via 0R selects R69 (fitted, holder) / R70 (DNP, eSIM). SMF05C pin2=GND to be confirmed at footprint verification."
- note removed: "VBAT_MODEM: 2x100uF + 1uF + 100nF + SMF5.0A, place <=5mm from U1 VBAT pads (57-60)."
Changed lines of the file:
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@@
 		)
 	)
-	(text "VBAT_MODEM: 2x100uF + 1uF + 100nF + SMF5.0A, place <=5mm from U1 VBAT pads (57-60)."
+	(text "VBAT_MODEM: 4x47uF X7R (F-13) + 1uF + 100nF + SMF5.0A, place <=5mm from U1 VBAT pads (57-60)."
 		(exclude_from_sim no)
 		(at 63.5 40.64 0)
@@
 		)
 	)
-	(text "U8 TXB0104: A=1.8V (VDD_EXT), B=3V3. A1<->B1 carries MCU TX -> modem MAIN_RXD(68); A2<->B2 modem MAIN_TXD(67) -> MCU RX; A3 RI(62); A4 DTR(66). OE held low until VDD_EXT rises."
+	(text "U8 TXB0104: A=1.8V (VDD_EXT), B=3V3. A1<->B1 carries MCU TX -> modem MAIN_RXD(68); A2<->B2 modem MAIN_TXD(67) -> MCU RX; A3 RI(62); A4 DTR(66). OE = 10k/100k from VDD_EXT (1.64 V)."
 		(exclude_from_sim no)
 		(at 203.2 38.1 0)
@@
 		(at 309.88 157.48)
 	)
-	(text "USIM: 33R series on DATA/CLK/RST, 100nF on VDD, SMF05C at the holder. MFF2 eSIM pads (X2, DNP) parallel; VDD via 0R selects R69 (fitted, holder) / R70 (DNP, eSIM). SMF05C pin2=GND to be confirmed at footprint verification."
+	(wire
+		(pts
+			(xy 381 72.39) (xy 381 68.58)
+		)
+		(stroke
+			(width 0)
+			(type default)
+		)
+	)
+	(label "VDD_EXT_1V8"
+		(at 381 68.58 90)
+		(effects
+			(font
+				(size 1.27 1.27)
+			)
+			(justify left bottom)
+		)
+	)
+	(wire
+		(pts
+			(xy 381 80.01) (xy 381 83.82)
+		)
+		(stroke
+			(width 0)
+			(type default)
+		)
+	)
+	(label "USIM_DET"
+		(at 381 83.82 270)
+		(effects
+			(font
+				(size 1.27 1.27)
+			)
+			(justify right bottom)
+		)
+	)
+	(text "USIM: 33R series on DATA/CLK/RST, 100nF on VDD, PESD5V0L5UY (19pF) at the holder, 51k USIM_DET pull-up to VDD_EXT. MFF2 eSIM pads (X2, DNP) parallel; VDD via 0R selects R69 (fitted, holder) / R70 (DNP, eSIM)."
 		(exclude_from_sim no)
 		(at 287.02 185.42 0)
@@
 			)
 		)
-		(property "LCSC" "C15849"
+		(property "LCSC" "C106858"
 			(at 101.6 50.8 0)
 			(hide yes)
@@
 			)
 		)
-		(property "LCSC" "C17407"
+		(property "LCSC" "C149504"
 			(at 30.48 88.9 0)
 			(hide yes)
@@
 			)
 		)
-		(property "Value" "10k"
+		(property "Value" "100k"
 			(at 226.06 91.44 0)
 			(effects
@@
 			)
 		)
-		(property "LCSC" "C17414"
+		(property "LCSC" "C149504"
 			(at 226.06 96.52 0)
 			(hide yes)
@@
 			)
 		)
-		(property "Value" "47k"
+		(property "Value" "10k"
 			(at 213.36 60.96 0)
 			(effects
@@
 			)
 		)
-		(property "LCSC" "C17713"
+		(property "LCSC" "C17414"
 			(at 213.36 66.04 0)
 			(hide yes)
@@
 			)
 		)
-		(property "LCSC" "C15849"
+		(property "LCSC" "C106858"
 			(at 213.36 50.8 0)
 			(hide yes)
@@
 			)
 		)
-		(property "Value" "SMF05C"
+		(property "Value" "PESD5V0L5UY"
 			(at 294.64 160.02 0)
 			(effects
@@
 			)
 		)
-		(property "LCSC" "C15879"
+		(property "LCSC" "C179747"
 			(at 294.64 165.1 0)
 			(hide yes)
@@
 					(unit 1)
 				)
+			)
+		)
+	)
+	(symbol
+		(lib_id "Device:R")
+		(at 381 76.2 0)
+		(unit 1)
+		(exclude_from_sim no)
+		(in_bom yes)
+		(on_board yes)
+		(dnp no)
+		(fields_autoplaced yes)
+		(property "Reference" "R91"
+			(at 381 73.66 0)
+			(effects
+				(font
+					(size 1.27 1.27)
+				)
+			)
+		)
+		(property "Value" "51k"
+			(at 381 71.12 0)
+			(effects
+				(font
+					(size 1.27 1.27)
+				)
+			)
+		)
+		(property "Footprint" "Resistor_SMD:R_0603_1608Metric"
+			(at 381 76.2 0)
+			(hide yes)
+			(effects
+				(font
+					(size 1.27 1.27)
+				)
+			)
+		)
+		(property "Datasheet" "~"
+			(at 381 76.2 0)
+			(hide yes)
+			(effects
+				(font
+					(size 1.27 1.27)
+				)
+			)
+		)
+		(property "LCSC" "C23196"
+			(at 381 76.2 0)
+			(hide yes)
+			(effects
+				(font
+					(size 1.27 1.27)
+				)
+			)
+		)
+		(pin "1"
+		)
+		(pin "2"
+		)
+		(instances
+			(project "telematics-tracker"
+				(path "/784bc421-9fc7-43cb-bfc3-562714cb3f68/70fac1b9-7bfc-5985-a8dc-ae866bd73e38"
+					(reference "R91")
+					(unit 1)
+				)
