File: telematics-tracker.kicad_pcb (KiCad board)
At the start: 4 copper layers, 82 x 62 mm, 216 parts, among them J1 WAFER-MX3.0-12PZZ, J2 B3B-XH-A, Q1 AM2390N-TP, Q10 MMBT3904, Q11 MMBT3904, Q12 MMBT3904, Q13 MMBT3906, Q14 MMBT3904, Q2 AM2390N-TP, Q3 AO3401A, Q4 MMBT3904, Q5 MMBT3904, Q6 MMBT3904, Q7 MMBT3904, Q8 MMBT3904, Q9 MMBT3904, U1 EC200UCNAA-N05-SGNSA, U2 AT32F403ACGT7, U3 QMI8658B, U4 SIT1051AT/3, U5 EG11752, U6 BQ25606RGER, U7 GD25Q64ESIGR, U8 TXB0104PWR, U9 ME6211C33M5G, X1 NANO-SIM, X2 MFF2-eSIM-pads, Y1 8MHz, Y2 32.768kHz

Commit message: F-24 defect fix: pi-shunt tap vias did not touch the ANT runs
The C48/C50 B.Cu stub tap vias sat 1.59/1.02 mm below their runs' short
verticals - the only two unconnected RF edges on the routed board. Generator
now emits the F.Cu extension from via to run vertex (SHUNTS carries run_y);
the same two locked segments were applied to the live board (corridors
verified empty first). T-stub discontinuity at the DNP option position was
already accepted under F-24; flag stays open for milestone-5 RF review.
Board: 108 unconnected, 0 errors.

Co-Authored-By: Claude Fable 5 <noreply@anthropic.com>
Routing:
- net /modem_rf/ANT_MAIN_M: track 3.76 -> 5.35 mm
- net /modem_rf/ANT_GNSS_M: track 3.61 -> 4.63 mm
Changed lines of the file:
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@@
 	(segment
 		(start 33.8996 45.4275)
-		(end 33.8996 47.2187)
+		(end 32.7628 45.4275)
 		(width 0.2)
 		(layer "B.Cu")
@@
 	(segment
 		(start 33.8996 45.4275)
-		(end 32.7628 45.4275)
+		(end 33.8996 47.2187)
 		(width 0.2)
 		(layer "B.Cu")
@@
 	(segment
 		(start 35.55 23.95)
-		(end 35.45 24.05)
+		(end 35.55 26.85)
 		(width 0.5)
 		(layer "B.Cu")
@@
 	(segment
 		(start 35.55 23.95)
-		(end 35.55 26.85)
+		(end 35.45 24.05)
 		(width 0.5)
 		(layer "B.Cu")
@@
 	(segment
 		(start 5.15 11.15)
-		(end 5.15 16.45)
+		(end 4.55 11.15)
 		(width 0.5)
 		(locked yes)
@@
 	(segment
 		(start 5.15 11.15)
-		(end 4.55 11.15)
+		(end 5.15 16.45)
 		(width 0.5)
 		(locked yes)
@@
 	(segment
 		(start 26.13 40.82)
-		(end 26.13 42.2042)
+		(end 27.7625 40.82)
 		(width 0.5)
 		(layer "F.Cu")
@@
 	(segment
 		(start 26.13 40.82)
-		(end 27.7625 40.82)
+		(end 26.13 42.2042)
 		(width 0.5)
 		(layer "F.Cu")
@@
 	(segment
 		(start 27.85 54.4)
-		(end 27.85 54.15)
+		(end 27.74 54.29)
 		(width 0.5)
 		(layer "F.Cu")
@@
 	(segment
 		(start 27.85 54.4)
-		(end 27.74 54.29)
+		(end 27.85 54.15)
 		(width 0.5)
 		(layer "F.Cu")
@@
 	(segment
 		(start 28.65 11.75)
-		(end 28.65 11.55)
+		(end 24.65 15.75)
 		(width 0.5)
 		(locked yes)
@@
 	(segment
 		(start 28.65 11.75)
-		(end 24.65 15.75)
+		(end 28.65 11.55)
 		(width 0.5)
 		(locked yes)
@@
 	(segment
 		(start 29.445 53.15)
-		(end 29.5 53.205)
+		(end 29.65 53.15)
 		(width 0.5)
 		(layer "F.Cu")
@@
 	(segment
 		(start 29.445 53.15)
-		(end 29.65 53.15)
+		(end 29.5 53.205)
 		(width 0.5)
 		(layer "F.Cu")
@@
 	(segment
 		(start 31.5 32.8)
-		(end 31.35 32.65)
+		(end 31.5 33.775)
 		(width 0.5)
 		(layer "F.Cu")
@@
 	(segment
 		(start 31.5 32.8)
-		(end 31.5 33.775)
+		(end 31.35 32.65)
 		(width 0.5)
 		(layer "F.Cu")
@@
 	(segment
 		(start 38.9927 30.2677)
-		(end 38.6729 30.2677)
+		(end 38.9927 29.0773)
 		(width 0.5)
 		(layer "F.Cu")
@@
 	(segment
 		(start 38.9927 30.2677)
-		(end 38.9927 29.0773)
+		(end 38.6729 30.2677)
 		(width 0.5)
 		(layer "F.Cu")
@@
 	)
 	(segment
+		(start 78.6 21.6)
+		(end 78.6 23.19)
+		(width 0.4)
+		(locked yes)
+		(layer "F.Cu")
+		(net "/modem_rf/ANT_MAIN_M")
+	)
+	(segment
 		(start 78.6 23.1925)
 		(end 78.6 23.389125)
@@
 	)
 	(segment
+		(start 78.6 27.3)
+		(end 78.6 28.32)
+		(width 0.4)
+		(locked yes)
+		(layer "F.Cu")
+		(net "/modem_rf/ANT_GNSS_M")
+	)
+	(segment
 		(start 78.6 28.321575)
 		(end 79.14 28.23)
@@
 	(segment
 		(start 26.5757 50.408)
-		(end 26.5757 52.9057)
+		(end 25.6935 49.5258)
 		(width 0.2)
 		(layer "In2.Cu")
@@
 	(segment
 		(start 26.5757 50.408)
-		(end 25.6935 49.5258)
+		(end 26.5757 52.9057)
 		(width 0.2)
 		(layer "In2.Cu")
@@
 	(segment
 		(start 50.8504 9.3985)
-		(end 51.4768 9.3985)
+		(end 50.7221 9.5268)
 		(width 0.2)
 		(layer "In2.Cu")
@@
 	(segment
 		(start 50.8504 9.3985)
-		(end 50.7221 9.5268)
+		(end 51.4768 9.3985)
 		(width 0.2)
 		(layer "In2.Cu")
@@
 	(segment
 		(start 68.6767 53.2666)
-		(end 68.6767 54.1421)
+		(end 73.5529 53.2666)
 		(width 0.2)
 		(layer "In2.Cu")
@@
 	(segment
 		(start 68.6767 53.2666)
-		(end 73.5529 53.2666)
+		(end 68.6767 54.1421)
 		(width 0.2)
 		(layer "In2.Cu")

Commit message: Pocket relief 1: six unrouted test points moved to the open B-side field east of x44
TP1/TP2/TP3/TP5/TP6/TP27 sat inside the congested x19-42 pocket where each
cost more wall than its short edge saved (gate-5 report). Moves applied to
the live board (courtyard + point-to-segment copper checks; only nets with
no routed copper were touched, 2 dangling MODEM_TX stubs ripped) and
mirrored into pcbplace anchors. Board: 109 unconnected, 0 errors.

Co-Authored-By: Claude Fable 5 <noreply@anthropic.com>
Parts:
- TP1, TP2, TP27, TP5: moved to B.Cu
- moved TP5 34.4 mm to (56.0, 26.0), turned to 180 degrees
- moved TP3 26.4 mm to (52.0, 26.0)
- moved TP6 25.3 mm to (46.0, 26.0)
- moved TP1 23.1 mm to (54.0, 22.0), turned to 180 degrees
- moved TP2 22.8 mm to (58.0, 22.0), turned to 180 degrees
- moved TP27 13.0 mm to (54.0, 40.0), turned to 180 degrees
Routing:
- net MODEM_TX: track 23.7 -> 22.1 mm

Commit message: LV rip-retry negotiation + TP re-site into the legal band
- Child --rip mode: textual local rip (4 mm around the starved net's pads,
  unlocked+unprotected only; board.Remove poisons SWIG on Py3.14, and
  LoadBoard needs the .kicad_pcb extension), starved net routes first,
  ripped signal nets re-route in the same child, pour nets requeue via
  REQUEUE lines. All-or-nothing: failures exit unsaved.
- Parent schedules one rip-retry per failing net from its measured pocket
  walls (top-3 unlocked, unprotected wall nets).
- TP1/TP2/TP3/TP5/TP27 re-sited into x43-50.5: the first move landed 5 of 6
  inside the LV router's own U1 via-field no-go (x51.4-70.5 y17.6-40.4) -
  legal copper, unroutable region. Spot checker now tests no-go rects and
  point-to-segment copper distance.

Co-Authored-By: Claude Fable 5 <noreply@anthropic.com>
Parts:
- moved TP27 16.8 mm to (49.0, 24.0)
- moved TP2 10.3 mm to (49.0, 27.0)
- moved TP1 9.90 mm to (47.0, 29.0)
- moved TP3 9.62 mm to (43.5, 21.5)
- moved TP5 9.30 mm to (48.5, 31.5)
Changed lines of the file:
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@@
 	(footprint "TestPoint_Pad_D1.5mm"
 		(layer "B.Cu")
-		(at 54 22 180)
+		(at 47 29 180)
 		(descr "SMD pad as test Point, diameter 1.5mm")
 		(tags "test point SMD pad")
@@
 	(footprint "TestPoint_Pad_D1.5mm"
 		(layer "B.Cu")
-		(at 58 22 180)
+		(at 49 27 180)
 		(descr "SMD pad as test Point, diameter 1.5mm")
 		(tags "test point SMD pad")
@@
 	(footprint "TestPoint_Pad_D1.5mm"
 		(layer "B.Cu")
-		(at 54 40 180)
+		(at 49 24 180)
 		(descr "SMD pad as test Point, diameter 1.5mm")
 		(tags "test point SMD pad")
@@
 	(footprint "TestPoint_Pad_D1.5mm"
 		(layer "B.Cu")
-		(at 52 26 180)
+		(at 43.5 21.5 180)
 		(descr "SMD pad as test Point, diameter 1.5mm")
 		(tags "test point SMD pad")
@@
 	(footprint "TestPoint_Pad_D1.5mm"
 		(layer "B.Cu")
-		(at 56 26 180)
+		(at 48.5 31.5 180)
 		(descr "SMD pad as test Point, diameter 1.5mm")
 		(tags "test point SMD pad")
@@
 	(segment
 		(start 35.55 23.95)
-		(end 35.55 26.85)
+		(end 35.45 24.05)
 		(width 0.5)
 		(layer "B.Cu")
@@
 	(segment
 		(start 35.55 23.95)
-		(end 35.45 24.05)
+		(end 35.55 26.85)
 		(width 0.5)
 		(layer "B.Cu")
@@
 	(segment
 		(start 29.445 53.15)
-		(end 29.5 53.205)
+		(end 29.65 53.15)
 		(width 0.5)
 		(layer "F.Cu")
@@
 	(segment
 		(start 29.445 53.15)
-		(end 29.65 53.15)
+		(end 29.5 53.205)
 		(width 0.5)
 		(layer "F.Cu")
