File: io.kicad_sch (KiCad schematic)
At the start: 68 parts, among them J1 WAFER-MX3.0-12PZZ, Q1 AM2390N-TP, Q2 AM2390N-TP, Q5 MMBT3904, Q6 MMBT3904, Q7 MMBT3904, Q8 MMBT3904, U4 SIT1051AT/3

Commit message: M3: F-9 review package, firmware notes, R80 pulse analysis, rules 1-9 audit, M4 prep
- docs/f9-review.md: all 76 NEEDS-HUMAN pins, 3-source verdicts (62 AGREE /
  14 CONFLICT flagged), GND + RESERVED rows first, nothing connected.
- docs/firmware-notes.md: FW-1..FW-17 + BV-1..BV-4.
- R80: selected FRP2512J100 C3013385 (2W); pulse duty computed at 8.5 mJ /
  384 W pk / tau 44 us per full-rated SMDJ strike (energy R-independent).
  F-15 NEW: 10R has NO load-line solution at the 10.5 V floor at full load -
  brown-out; recommend 1R FRS2512F1R00TS C55348540 (anti-surge). Decision gate.
- Rules audit: 1 NOT MET (F-13 X5R/6.3V modem bulk caps), 8 NOT MET (F-14
  six missing TPs: VIN, VBAT_MODEM, CANH/CANL, modem UART), rest MET/N-A
  with evidence; section-6 blocks all MET as amended.
- M4 prep: stackup defined (L1 sig/RF, L2 solid GND, L3 power, L4 sig,
  JLC7628 1.6mm); docs/placement-study.svg on PROVISIONAL 80x60 outline.
- Footprint checks: J1 posts RESOLVED (derived footprint with 2x NPTH from
  XUNPU drawing, J1 re-pointed); SIM pad map VERIFIED but posts missing ->
  F-16 (y-datum ambiguous, no copper guessed); SMF05C pin2=GND VERIFIED
  (onsemi pin table) - caveat closed; X2 remapped to authoritative ETSI/
  1GLOBAL MFF2 pinout (old 6-pin placeholder was wrong), land pattern gated
  F-17 on vendor packaging spec.

ERC 0 errors / 14 justified warnings; checkpins 48/48 + F-10 8/8 PASS.

Co-Authored-By: Claude Fable 5 <noreply@anthropic.com>
Parts:
- J1: footprint Connector_Molex:Molex_Micro-Fit_3.0_43045-1212_2x06_P3.00mm_Vertical -> jlc:XUNPU_MX3.0-12PZZ_2x06_P3.00mm_Vertical
Changed lines of the file:
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@@
 			)
 		)
-		(property "Footprint" "Connector_Molex:Molex_Micro-Fit_3.0_43045-1212_2x06_P3.00mm_Vertical"
+		(property "Footprint" "jlc:XUNPU_MX3.0-12PZZ_2x06_P3.00mm_Vertical"
 			(at 58.42 101.6 0)
 			(hide yes)

Commit message: M3 close: F-15 R80 1R, F-14 six test points, ambient rating, CPWG geometry
F-15: R80 10R (C3013385) -> 1R anti-surge FRS2512F1R00TS (C55348540).
At the 10.5 V floor and full load the 10R version had NO load-line solution:
V_B^2 - 9.8*V_B + 59 = 0, discriminant -140. Max power transfer through 10R
from 9.8 V is V^2/4R = 2.4 W against a 5.9 W demand - a hard brown-out. At 1R:
V_B = 9.16 V, I = 0.644 A, 0.41 W worst-case continuous, 24 W ceiling.
Pulse energy unchanged at 8.5 mJ (E = CdV^2/2 is independent of R) but peak
goes 384 W -> 3.8 kW and tau 44 us -> 4.4 us, which is why the part must be
anti-surge rather than plain thick film. Confirming that pulse curve joins F-12
on the bench list.

F-14: TP23 VIN, TP24 VBAT_MODEM, TP25 CANH, TP26 CANL, TP27 MODEM_TX,
TP28 MODEM_RX. Each verified against the netlist to share its net with the
real circuit nodes. hier() used for hierarchical nets and net() only for
sheet-local ones, so ERC stayed at exactly 0 errors / 14 warnings with no new
same_local_global_label entries. Rule 8 now MET (28 test points).

Product spec: rated operating ambient -20 to +70 C, housing shaded or
light-coloured, 85 C survival not operating - added to handoff section 1.1 and
a new docs/installation-sheet.md. Governed by U1: EC200U V1.2 Table 42 p.75
gives operating -35..+75 C (meets 3GPP) and extended -40..+85 C (functions
maintained but Pout may exceed 3GPP tolerances), so +70 C keeps 5 C to the
compliant limit and 85 C is exactly the extended limit.

NEW FLAG F-19: typical 1S Li-ion is -20..+60 C discharge, narrower than the
+70 C product ceiling. Charging is already protected by the BQ25606 JEITA
network; discharge above 60 C and calendar ageing are not. Decision needed -
accept with a shorter battery service interval, or narrow the rating to +60 C.

M4 input: 50 ohm CPWG for JLC7628 L1-L2 computed via Ghione-Naldi conformal
mapping (elliptic integrals by AGM), cross-checked against Hammerstad-Jensen
microstrip. h = 0.2104 mm (1x 7628 prepreg). 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
Parts:
- added TP25: CANH, TestPoint:TestPoint_Pad_D1.5mm, symbol Connector:TestPoint
- added TP26: CANL, TestPoint:TestPoint_Pad_D1.5mm, symbol Connector:TestPoint
Connections:
- net CANH: now also TP25.1
- net CANL: now also TP26.1
Other:
- note added: "F-14 test points: CANH / CANL at the connector side of L2."
Changed lines of the file:
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@@
+	(wire
+		(pts
+			(xy 30.48 271.78) (xy 30.48 276.86)
+		)
+		(stroke
+			(width 0)
+			(type default)
+		)
+	)
+	(label "CANH"
+		(at 30.48 276.86 270)
+		(effects
+			(font
+				(size 1.27 1.27)
+			)
+			(justify right bottom)
+		)
+	)
+	(wire
+		(pts
+			(xy 45.72 271.78) (xy 45.72 276.86)
+		)
+		(stroke
+			(width 0)
+			(type default)
+		)
+	)
+	(label "CANL"
+		(at 45.72 276.86 270)
+		(effects
+			(font
+				(size 1.27 1.27)
+			)
+			(justify right bottom)
+		)
+	)
+	(text "F-14 test points: CANH / CANL at the connector side of L2."
+		(exclude_from_sim no)
+		(at 30.48 264.16 0)
+		(effects
+			(font
+				(size 1.27 1.27)
+			)
+			(justify left bottom)
+		)
+	)
 	(wire
 		(pts
@@
 					(unit 1)
 				)
+			)
+		)
+	)
+	(symbol
+		(lib_id "Connector:TestPoint")
+		(at 30.48 271.78 0)
+		(unit 1)
+		(exclude_from_sim no)
+		(in_bom yes)
+		(on_board yes)
+		(dnp no)
+		(fields_autoplaced yes)
+		(property "Reference" "TP25"
+			(at 30.48 269.24 0)
+			(effects
+				(font
+					(size 1.27 1.27)
+				)
+			)
+		)
+		(property "Value" "CANH"
+			(at 30.48 266.7 0)
+			(effects
+				(font
+					(size 1.27 1.27)
+				)
+			)
+		)
+		(property "Footprint" "TestPoint:TestPoint_Pad_D1.5mm"
+			(at 30.48 271.78 0)
+			(hide yes)
+			(effects
+				(font
+					(size 1.27 1.27)
+				)
+			)
+		)
+		(property "Datasheet" "~"
+			(at 30.48 271.78 0)
+			(hide yes)
+			(effects
+				(font
+					(size 1.27 1.27)
+				)
+			)
+		)
+		(pin "1"
+		)
+		(instances
+			(project "telematics-tracker"
+				(path "/784bc421-9fc7-43cb-bfc3-562714cb3f68/cbd713bf-4a1d-56fd-a164-2267d4bf4daf"
+					(reference "TP25")
+					(unit 1)
+				)
+			)
+		)
+	)
+	(symbol
+		(lib_id "Connector:TestPoint")
+		(at 45.72 271.78 0)
+		(unit 1)
+		(exclude_from_sim no)
+		(in_bom yes)
+		(on_board yes)
+		(dnp no)
+		(fields_autoplaced yes)
+		(property "Reference" "TP26"
+			(at 45.72 269.24 0)
+			(effects
+				(font
+					(size 1.27 1.27)
+				)
+			)
+		)
+		(property "Value" "CANL"
+			(at 45.72 266.7 0)
+			(effects
+				(font
+					(size 1.27 1.27)
+				)
+			)
+		)
+		(property "Footprint" "TestPoint:TestPoint_Pad_D1.5mm"
+			(at 45.72 271.78 0)
+			(hide yes)
+			(effects
+				(font
+					(size 1.27 1.27)
+				)
+			)
+		)
+		(property "Datasheet" "~"
+			(at 45.72 271.78 0)
+			(hide yes)
+			(effects
+				(font
+					(size 1.27 1.27)
+				)
+			)
+		)
+		(pin "1"
+		)
+		(instances
+			(project "telematics-tracker"
+				(path "/784bc421-9fc7-43cb-bfc3-562714cb3f68/cbd713bf-4a1d-56fd-a164-2267d4bf4daf"
+					(reference "TP26")
+					(unit 1)
+				)

Commit message: Step 1-3: fix rule floors, classify SW_BUCK as HV, shrink, fix HV router
Step 1 - rule mismatch fixed and verified:
  netclasses.py gains BOARD_RULES + _assert_floors(). Every class now meets
  track >= 0.20 mm and via annulus >= 0.10 mm. min_clearance had been silently
  reset to 0.0 by a KiCad round trip; restored to 0.15 and now asserted after
  the round trip so it cannot regress unnoticed. Exported DSN verified to carry
  the values (kicad_default 200, GND 500, MODEM_BULK 2000, RF 400, HV 500/600).

Step 2 - HV hand-routing, and three real defects it uncovered:

  1. /power/SW_BUCK was in the Default netclass. It is the buck switching node:
     it swings from GND to VIN every cycle, so it is a 100 V net with fast
     edges, and it was running at 0.20 mm track / 0.15 mm clearance. U5_VB
     (bootstrap) rides on it and was equally misclassified. Both moved to HV.
     Found because the maze router treated SW_BUCK as LV and threw a 1.50 mm
     halo around U5's own VIN pins, making /power/VIN_B unroutable at 0/4.

  2. HV_ZONE stopped at x = 20.0 and so EXCLUDED the buck primary side. U5 sits
     at x 35.4..42.3 with C73, C74 and D16 beside it, and VIN_B runs 22 mm from
     R80 to reach it. The highest-energy node on the board was outside the HV
     rule area - which also meant the U5 package exception approved under F-20
     was dead code, since it is conditioned on insideArea('HV_ZONE'). HV_ZONE
     is now L-shaped: left strip plus the buck primary.

  3. Three defects in pcbroute_hv.py itself, together responsible for 128 of
     the 129 clearance violations the first routed board had:
       - halos were sized for a 0.50 mm track (half 0.25) but the router also
         drops 0.80 mm vias, so cells legal for a track were illegal for a via
       - halo extents were quantised with round(), letting a cell centre sit up
         to RES/2 = 0.075 mm inside the forbidden region. That is exactly the
         size of the 0.545..0.594 mm shortfalls DRC reporte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
Parts:
- removed C30: 100nF, Capacitor_SMD:C_0603_1608Metric, symbol Device:C
- removed R40: 100k, Resistor_SMD:R_0805_2012Metric, symbol Device:R
- removed R41: 9.1k, Resistor_SMD:R_0805_2012Metric, symbol Device:R
- removed TP10: VIN_SENSE, TestPoint:TestPoint_Pad_D1.5mm, symbol Connector:TestPoint
- removed TP11: IGN_SENSE, TestPoint:TestPoint_Pad_D1.5mm, symbol Connector:TestPoint
- removed TP12: VBAT_SENSE, TestPoint:TestPoint_Pad_D1.5mm, symbol Connector:TestPoint
- removed TP8: J1_SPARE1, TestPoint:TestPoint_Pad_D1.5mm, symbol Connector:TestPoint
- removed TP9: J1_SPARE2, TestPoint:TestPoint_Pad_D1.5mm, symbol Connector:TestPoint
Other:
- note removed: "Spare ADC divider footprint - fitted DNP (handoff section 5, PB1)."

Commit message: BOM verification (milestone 5): 28 wrong or unverified lines fixed against LCSC/JLCPCB data; F-5 and F-22 closed
Wrong values (C1/C2 22pF for 18pF, C3/C4, R56/R58 10k for 47k, R66-R68
100R for 33R), wrong packages (C12/C63, C83, R71/R72, Y1 5032 on a 3225
footprint), Y2 12.5pF crystal on 6.8pF caps (now a 7pF FC-135), red LED
number on the green and blue LEDs (R4/R6 330R for their Vf), a
non-existent C-number (2.2k), and nine TBD placeholders.

tools/bom_audit.py: value / voltage / package / LED colour / crystal load /
stock (JLCPCB and LCSC) per line -> docs/bom-audit.md, out/bom-mpn.csv
(manufacturer + MPN). Netlist connectivity unchanged, ERC 0, checkpins ok.

Co-Authored-By: Claude Opus 5.5 <noreply@anthropic.com>
Parts:
- R45, R49: LCSC C4356 -> C17520
Changed lines of the file:
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@@
 			)
 		)
-		(property "LCSC" "C4356"
+		(property "LCSC" "C17520"
 			(at 121.92 259.08 0)
 			(hide yes)
@@
 			)
 		)
-		(property "LCSC" "C4356"
+		(property "LCSC" "C17520"
 			(at 121.92 304.8 0)
 			(hide yes)

Commit message: Pre-order verification review: 12 would-fail faults fixed, report added
Schematic (tools/sheets.py, sheets regenerated):
- D2 SMDJ100A: D_Zener symbol, cathode to VIN_P (was drawn forward with
  the bidirectional D_TVS symbol)
- D10/D11 BAV99 clamps: pin 1 (anode) GND, pin 2 (cathode) 3V3 (KiCad's
  hidden K/A/K pin names contradict the Nexperia pinout)
- D5/D6: BAV70 common-cathode replaces the mirrored BAV99 (opto LED was
  bypassed)
- U8 TXB0104 OE: 10k/100k = 1.64 V (47k/10k gave 0.32 V, UART disabled)
- R82 0.1R: EG11752 2 A peak limit (0R disabled it)
- D7/D8 flyback cathodes to VIN_P behind D1 (reverse-polarity path via
  the Q1/Q2 body diodes), VIN_P exported as a hierarchical net
- Q1/Q2 gate pulldown 100k (4.89 V; 10k gave 4.07 V), DI pull-up 220k,
  R91 51k USIM_DET pull-up, PESD5V0L5UY SIM ESD, X7R 1uF/4.7uF, 100k
  C149504, comments and notes corrected

Board (DRC-gated routes via tools/manual_routes.py + tools/board_fixes.py):
- D2/D10/D11 turned, NRST via moved, VIN trunk re-laid around D7/D8,
  VIN_P B.Cu run to D1, R91 on B.Cu, VBAT_BT 0.6 mm F.Cu to J2, SW_CHG
  0.4 mm, PMID 0.3/0.5 mm, DNP flags, C61<->C80 swap, 28 RF stitching
  vias, 9 vias under U5's pad; values updated
- manual_routes: delvia/padnet/rotate/value/move ops, ACCEPT_EQUAL

Checks: parity 0 mismatches (212 parts, 727 pad nets), ERC 0 errors,
pin checklist pass, DRC 0 errors / 0 unconnected, BOM audit 76/76 clean.

Docs: firmware-notes FW-6/8/13/14/17 + FW-18..22, BV-1/5/6/7; handoff and
installation sheet corrected (12 V floor, DI not isolated, values);
design-log entry; docs/verification-report.pdf (OK / NOT OK per item).

Co-Authored-By: Claude Fable 5.1 <noreply@anthropic.com>
Parts:
- D5, D6: value BAV99 -> BAV70; symbol Diode:BAV99 -> Diode:BAV70; LCSC C2500 -> C2501
- R21, R22: value 47k -> 220k; LCSC C17713 -> C17556
- R25, R26: value 10k -> 100k; LCSC C17414 -> C149504
- R30, R31, R32, R33, R34, R35: LCSC C17407 -> C149504
Connections:
- net 3V3: now also D10.2 (A), D11.2 (A); no longer D10.1 (K), D11.1 (K)
- net GND: now also D10.1 (K), D11.1 (K); no longer D10.2 (A), D11.2 (A)
- net VIN: no longer D7.1 (K), D8.1 (K)
- new net VIN_P: D7.1 (K), D8.1 (K)
Other:
- note added: "DI1/DI2: 36k series (3x12k 1206, F-7) -> EL357N(D) opto, 220k pull-up + 100nF at the MCU side. Valid input 10.5-100 V."
- note added: "DO1/DO2 (F-10): two-stage NPN driver from 5V0, non-inverting, default OFF (base pulldown + QnB clamps gate; 100k gate pulldown -> 4.9 V VGS). SS3200 200V flyback to VIN_P, behind D1 (F-11, reverse-polarity review 2026-09-30). DO1/DO2 inactive on battery backup (5V0 absent)."
- note added: "MACHINE I/O - CAN, ground-referenced digital inputs, low-side outputs, supply sensing. HV zone: J1 / dividers / DI series R / DO drains."
- note added: "Valid DI input range 10.5-100 V. DO loads: relay coils / buzzers <= 0.5 A at 12/24 V."
- note removed: "DI1/DI2: 36k series (3x12k 1206, F-7) -> EL357N(D) opto, 47k pull-up + 100nF at the MCU side. Valid input 10.5-100 V."
- note removed: "DO1/DO2 (F-10): two-stage NPN driver from 5V0, non-inverting, default OFF (base pulldown + QnB clamps gate; 10k gate pulldown retained). SS3200 200V flyback to VIN (F-11). DO1/DO2 inactive on battery backup (5V0 absent)."
- note removed: "MACHINE I/O - CAN, isolated digital inputs, low-side outputs, supply sensing. HV zone: J1 / dividers / DI series R / DO drains."
- note removed: "Valid DI input range 9-100 V. DO loads: relay coils / buzzers <= 0.5 A at 12/24 V."
Changed lines of the file:
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@@
 	(generator_version "9.0")
 	(paper "A3")
-	(text "MACHINE I/O - CAN, isolated digital inputs, low-side outputs, supply sensing.  HV zone: J1 / dividers / DI series R / DO drains."
+	(text "MACHINE I/O - CAN, ground-referenced digital inputs, low-side outputs, supply sensing.  HV zone: J1 / dividers / DI series R / DO drains."
 		(exclude_from_sim no)
 		(at 25.4 20.32 0)
@@
 		)
 	)
-	(text "Valid DI input range 9-100 V.  DO loads: relay coils / buzzers <= 0.5 A at 12/24 V."
+	(text "Valid DI input range 10.5-100 V.  DO loads: relay coils / buzzers <= 0.5 A at 12/24 V."
 		(exclude_from_sim no)
 		(at 25.4 25.4 0)
@@
 		)
 	)
-	(text "DI1/DI2: 36k series (3x12k 1206, F-7) -> EL357N(D) opto, 47k pull-up + 100nF at the MCU side.  Valid input 10.5-100 V."
+	(text "DI1/DI2: 36k series (3x12k 1206, F-7) -> EL357N(D) opto, 220k pull-up + 100nF at the MCU side.  Valid input 10.5-100 V."
 		(exclude_from_sim no)
 		(at 81.28 157.48 0)
@@
 		)
 	)
-	(label "VIN"
+	(hierarchical_label "VIN_P"
+		(shape input)
 		(at 199.39 256.54 180)
 		(effects
@@
 				(size 1.27 1.27)
 			)
-			(justify right bottom)
+			(justify right)
 		)
 	)
@@
 		)
 	)
-	(label "VIN"
+	(hierarchical_label "VIN_P"
+		(shape input)
 		(at 199.39 302.26 180)
 		(effects
@@
 				(size 1.27 1.27)
 			)
-			(justify right bottom)
+			(justify right)
 		)
 	)
-	(text "DO1/DO2 (F-10): two-stage NPN driver from 5V0, non-inverting, default OFF (base pulldown + QnB clamps gate; 10k gate pulldown retained).  SS3200 200V flyback to VIN (F-11).  DO1/DO2 inactive on battery backup (5V0 absent)."
+	(text "DO1/DO2 (F-10): two-stage NPN driver from 5V0, non-inverting, default OFF (base pulldown + QnB clamps gate; 100k gate pulldown -> 4.9 V VGS).  SS3200 200V flyback to VIN_P, behind D1 (F-11, reverse-polarity review 2026-09-30).  DO1/DO2 inactive on battery backup (5V0 absent)."
 		(exclude_from_sim no)
 		(at 55.88 259.08 0)
@@
 	(wire
 		(pts
-			(xy 363.22 63.5) (xy 358.14 63.5)
+			(xy 363.22 63.5) (xy 359.41 63.5)
 		)
 		(stroke
@@
 		)
 	)
-	(label "3V3"
-		(at 358.14 63.5 180)
-		(effects
-			(font
-				(size 1.27 1.27)
-			)
-			(justify right bottom)
-		)
-	)
 	(wire
 		(pts
-			(xy 378.46 63.5) (xy 382.27 63.5)
+			(xy 378.46 63.5) (xy 383.54 63.5)
 		)
 		(stroke
@@
 		)
 	)
+	(label "3V3"
+		(at 383.54 63.5 0)
+		(effects
+			(font
+				(size 1.27 1.27)
+			)
+			(justify left bottom)
+		)
+	)
 	(wire
 		(pts
@@
 	(wire
 		(pts
-			(xy 363.22 106.68) (xy 358.14 106.68)
+			(xy 363.22 106.68) (xy 359.41 106.68)
 		)
 		(stroke
@@
 		)
 	)
-	(label "3V3"
-		(at 358.14 106.68 180)
-		(effects
-			(font
-				(size 1.27 1.27)
-			)
-			(justify right bottom)
-		)
-	)
 	(wire
 		(pts
-			(xy 378.46 106.68) (xy 382.27 106.68)
+			(xy 378.46 106.68) (xy 383.54 106.68)
 		)
 		(stroke
@@
 		)
 	)
+	(label "3V3"
+		(at 383.54 106.68 0)
+		(effects
+			(font
+				(size 1.27 1.27)
+			)
+			(justify left bottom)
+		)
+	)
 	(text "VIN and IGN sensing: 300k (3x100k 0805) : 9.1k, 100nF, BAV99 clamp to 3V3/GND.  IGN also serves as the EXTI wake input."
 		(exclude_from_sim no)
@@
 	)
 	(symbol
-		(lib_id "Diode:BAV99")
+		(lib_id "Diode:BAV70")
 		(at 121.92 190.5 0)
 		(unit 1)
@@
 			)
 		)
-		(property "Value" "BAV99"
+		(property "Value" "BAV70"
 			(at 121.92 185.42 0)
 			(effects
@@
 			)
 		)
-		(property "LCSC" "C2500"
+		(property "LCSC" "C2501"
 			(at 121.92 190.5 0)
 			(hide yes)
@@
 			)
 		)
-		(property "Value" "47k"
+		(property "Value" "220k"
 			(at 170.18 160.02 0)
 			(effects
@@
 			)
 		)
-		(property "LCSC" "C17713"
+		(property "LCSC" "C17556"
 			(at 170.18 165.1 0)
 			(hide yes)
@@
 	)
 	(symbol
-		(lib_id "Diode:BAV99")
+		(lib_id "Diode:BAV70")
 		(at 121.92 238.76 0)
 		(unit 1)
@@
 			)
 		)
-		(property "Value" "BAV99"
+		(property "Value" "BAV70"
 			(at 121.92 233.68 0)
 			(effects
@@
 			)
 		)
-		(property "LCSC" "C2500"
+		(property "LCSC" "C2501"
 			(at 121.92 238.76 0)
 			(hide yes)
@@
 			)
 		)
-		(property "Value" "47k"
+		(property "Value" "220k"
 			(at 170.18 208.28 0)
 			(effects
@@
 			)
 		)
-		(property "LCSC" "C17713"
+		(property "LCSC" "C17556"
 			(at 170.18 213.36 0)
 			(hide yes)
@@
 			)
 		)
-		(property "Value" "10k"
+		(property "Value" "100k"
 			(at 149.86 269.24 0)
 			(effects
@@
 			)
 		)
-		(property "LCSC" "C17414"
+		(property "LCSC" "C149504"
 			(at 149.86 274.32 0)
 			(hide yes)
@@
 			)
 		)
-		(property "Value" "10k"
+		(property "Value" "100k"
 			(at 149.86 314.96 0)
 			(effects
@@
 			)
 		)
-		(property "LCSC" "C17414"
+		(property "LCSC" "C149504"
 			(at 149.86 320.04 0)
 			(hide yes)
@@
 			)
 		)
-		(property "LCSC" "C17407"
+		(property "LCSC" "C149504"
 			(at 292.1 50.8 0)
 			(hide yes)
@@
 			)
 		)
-		(property "LCSC" "C17407"
+		(property "LCSC" "C149504"
 			(at 307.34 50.8 0)
 			(hide yes)
@@
 			)
 		)
-		(property "LCSC" "C17407"
+		(property "LCSC" "C149504"
 			(at 322.58 50.8 0)
 			(hide yes)
@@
 	(symbol
 		(lib_id "power:GND")
-		(at 382.27 63.5 0)
+		(at 359.41 63.5 0)
 		(unit 1)
 		(exclude_from_sim no)
@@
 		(fields_autoplaced yes)
 		(property "Reference" "#PWR058"
-			(at 382.27 55.88 0)
+			(at 359.41 55.88 0)
 			(effects
 				(font
@@
 		)
 		(property "Value" "GND"
-			(at 382.27 63.5 0)
+			(at 359.41 63.5 0)
 			(hide yes)
 			(effects
@@
 			)
 		)
-		(property "LCSC" "C17407"
+		(property "LCSC" "C149504"
 			(at 292.1 93.98 0)
 			(hide yes)
@@
 			)
 		)
-		(property "LCSC" "C17407"
+		(property "LCSC" "C149504"
 			(at 307.34 93.98 0)
 			(hide yes)
@@
 			)
 		)
-		(property "LCSC" "C17407"
+		(property "LCSC" "C149504"
 			(at 322.58 93.98 0)
 			(hide yes)
@@
 	(symbol
 		(lib_id "power:GND")
-		(at 382.27 106.68 0)
+		(at 359.41 106.68 0)
 		(unit 1)
 		(exclude_from_sim no)
@@
 		(fields_autoplaced yes)
 		(property "Reference" "#PWR061"
-			(at 382.27 99.06 0)
+			(at 359.41 99.06 0)
 			(effects
 				(font
@@
 		)
 		(property "Value" "GND"
-			(at 382.27 106.68 0)
+			(at 359.41 106.68 0)
 			(hide yes)
 			(effects
