File: io.kicad_sch (KiCad schematic)
At the start: 62 parts, among them J1 WAFER-MX3.0-12PZZ, Q1 AM2390N-TP, Q2 AM2390N-TP, Q5 MMBT3904, Q6 MMBT3904, Q7 MMBT3904, Q8 MMBT3904, U4 SIT1051AT/3

Commit message: Opto OK1/OK2 to the EL357N(D) bin (C42385002); India purchase BOM
C359074 is EL357N(A) (CTR 50-150 %); the DI pull-up margin was calculated
for the (D) bin (300-600 %), which JLCPCB stocks as C42385002. The audit
compares part families, not CTR bins - noted in the purchase list.

tools/bom_india.py: purchase list for buying parts in India from
out/bom-mpn.csv - plain "ask for" wording per line, exact part number,
substitute rule, source (local shop / distributor / LCSC-only / Quectel),
quantities for N boards with spares; CSV + printable PDF in docs/.

Package rebuilt: out/telematics-tracker-mfg-2026-09-30-86ea36c.zip

Co-Authored-By: Claude Fable 5.1 <noreply@anthropic.com>
Parts:
- OK1, OK2: LCSC C359074 -> C42385002
Changed lines of the file:
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@@
 			)
 		)
-		(property "LCSC" "C359074"
+		(property "LCSC" "C42385002"
 			(at 142.24 175.26 0)
 			(hide yes)
@@
 			)
 		)
-		(property "LCSC" "C359074"
+		(property "LCSC" "C42385002"
 			(at 142.24 223.52 0)
 			(hide yes)
