File: telematics-tracker.kicad_sch (KiCad schematic)
At the start: 0 parts

Commit message: Pre-order verification review: 12 would-fail faults fixed, report added
Schematic (tools/sheets.py, sheets regenerated):
- D2 SMDJ100A: D_Zener symbol, cathode to VIN_P (was drawn forward with
  the bidirectional D_TVS symbol)
- D10/D11 BAV99 clamps: pin 1 (anode) GND, pin 2 (cathode) 3V3 (KiCad's
  hidden K/A/K pin names contradict the Nexperia pinout)
- D5/D6: BAV70 common-cathode replaces the mirrored BAV99 (opto LED was
  bypassed)
- U8 TXB0104 OE: 10k/100k = 1.64 V (47k/10k gave 0.32 V, UART disabled)
- R82 0.1R: EG11752 2 A peak limit (0R disabled it)
- D7/D8 flyback cathodes to VIN_P behind D1 (reverse-polarity path via
  the Q1/Q2 body diodes), VIN_P exported as a hierarchical net
- Q1/Q2 gate pulldown 100k (4.89 V; 10k gave 4.07 V), DI pull-up 220k,
  R91 51k USIM_DET pull-up, PESD5V0L5UY SIM ESD, X7R 1uF/4.7uF, 100k
  C149504, comments and notes corrected

Board (DRC-gated routes via tools/manual_routes.py + tools/board_fixes.py):
- D2/D10/D11 turned, NRST via moved, VIN trunk re-laid around D7/D8,
  VIN_P B.Cu run to D1, R91 on B.Cu, VBAT_BT 0.6 mm F.Cu to J2, SW_CHG
  0.4 mm, PMID 0.3/0.5 mm, DNP flags, C61<->C80 swap, 28 RF stitching
  vias, 9 vias under U5's pad; values updated
- manual_routes: delvia/padnet/rotate/value/move ops, ACCEPT_EQUAL

Checks: parity 0 mismatches (212 parts, 727 pad nets), ERC 0 errors,
pin checklist pass, DRC 0 errors / 0 unconnected, BOM audit 76/76 clean.

Docs: firmware-notes FW-6/8/13/14/17 + FW-18..22, BV-1/5/6/7; handoff and
installation sheet corrected (12 V floor, DI not isolated, values);
design-log entry; docs/verification-report.pdf (OK / NOT OK per item).

Co-Authored-By: Claude Fable 5.1 <noreply@anthropic.com>
Other:
- sheet io ports: added VIN_P; removed none
- sheet power ports: added VIN_P; removed none
Changed lines of the file:
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@@
+	(wire
+		(pts
+			(xy 228.6 55.88) (xy 220.98 55.88)
+		)
+		(stroke
+			(width 0)
+			(type default)
+		)
+	)
+	(global_label "VIN_P"
+		(shape input)
+		(at 220.98 55.88 180)
+		(fields_autoplaced yes)
+		(effects
+			(font
+				(size 1.27 1.27)
+			)
+			(justify right)
+		)
+		(property "Intersheetrefs" "${INTERSHEET_REFS}"
+			(at 220.98 55.88 0)
+			(hide yes)
+			(effects
+				(font
+					(size 1.27 1.27)
+				)
+				(justify right)
+			)
+		)
+	)
 	(wire
 		(pts
@@
 		(property "Intersheetrefs" "${INTERSHEET_REFS}"
 			(at 17.78 162.56 0)
+			(hide yes)
+			(effects
+				(font
+					(size 1.27 1.27)
+				)
+				(justify right)
+			)
+		)
+	)
+	(wire
+		(pts
+			(xy 25.4 165.1) (xy 17.78 165.1)
+		)
+		(stroke
+			(width 0)
+			(type default)
+		)
+	)
+	(global_label "VIN_P"
+		(shape output)
+		(at 17.78 165.1 180)
+		(fields_autoplaced yes)
+		(effects
+			(font
+				(size 1.27 1.27)
+			)
+			(justify right)
+		)
+		(property "Intersheetrefs" "${INTERSHEET_REFS}"
+			(at 17.78 165.1 0)
 			(hide yes)
 			(effects
@@
 	(sheet
 		(at 228.6 25.4)
-		(size 44.45 33.02)
+		(size 44.45 35.56)
 		(fields_autoplaced yes)
 		(stroke
@@
 		)
 		(property "Sheetfile" "io.kicad_sch"
-			(at 228.6 59.82 0)
+			(at 228.6 62.36 0)
 			(effects
 				(font
@@
 		(pin "VIN" input
 			(at 228.6 53.34 180)
+			(effects
+				(font
+					(size 1.27 1.27)
+				)
+				(justify right)
+			)
+		)
+		(pin "VIN_P" input
+			(at 228.6 55.88 180)
 			(effects
 				(font
@@
 			(effects
 				(font
+					(size 1.27 1.27)
+				)
+				(justify right)
+			)
+		)
+		(pin "VIN_P" output
+			(at 25.4 165.1 180)
+			(effects
+				(font
