File: power.kicad_sch (KiCad schematic)
At the start: 42 parts, among them J2 B3B-XH-A, U5 EG11752, U6 BQ25606RGER, U9 ME6211C33M5G

Commit message: Fix split SYS rail; relief round 3 anchors; L3 pours redrawn to the pads
SCHEMATIC FAULT FIXED: the power sheet carried only LOCAL "SYS" labels, so
the charger output (U6.15/16, L3, C65/C66/C68, U9 input) was net /power/SYS
and never left the sheet, while the modem power switch (Q3, Q13, R52), the
battery-sense divider (R38) and TP13 sat on a global SYS with no source.
ERC reported it only as same_local_global_label (a "justified" warning).
U6.15 now carries a hierarchical label like 3V3/5V0 do; SYS is one net of
11 members. ERC 0 errors / 22 warnings (same two benign classes);
checkpins 48/48 still passes.

Placement (relief round 3, variant A of four parallel trials): U8 -> back
side (49.9, 47.0) beside X1/U1, its only partners; U7 -> back side
(46.9, 15.6), out of U2's west escape corridor. Variant A reached 92
unconnected after one hybrid cycle from a fresh regeneration (floor was 109).

L3 pours: measured on the routed board, the old "5V0" band y 27.5-39 held
14 3V3 pads and 4 5V0 pads, the "SYS" band held 5 of the 5V0 pads, and the
north "3V3 finger" held no 3V3 pad - so pour-taps were impossible for most
power pads. 3V3 is now the background pour of the LV area; 5V0 and SYS get
tight priority-1 islands computed by a greedy no-foreign-pad search
(13/16 5V0 pads, 9/13 SYS pads covered; no 3V3 pad lands in a foreign
island). VBAT_MODEM keeps its island at priority 1.

Co-Authored-By: Claude Fable 5.1 <noreply@anthropic.com>
Changed lines of the file:
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@@
 		)
 	)
-	(label "SYS"
+	(hierarchical_label "SYS"
+		(shape output)
 		(at 130.81 200.66 0)
 		(effects
@@
 				(size 1.27 1.27)
 			)
-			(justify left bottom)
+			(justify left)
 		)
 	)

Commit message: BOM verification (milestone 5): 28 wrong or unverified lines fixed against LCSC/JLCPCB data; F-5 and F-22 closed
Wrong values (C1/C2 22pF for 18pF, C3/C4, R56/R58 10k for 47k, R66-R68
100R for 33R), wrong packages (C12/C63, C83, R71/R72, Y1 5032 on a 3225
footprint), Y2 12.5pF crystal on 6.8pF caps (now a 7pF FC-135), red LED
number on the green and blue LEDs (R4/R6 330R for their Vf), a
non-existent C-number (2.2k), and nine TBD placeholders.

tools/bom_audit.py: value / voltage / package / LED colour / crystal load /
stock (JLCPCB and LCSC) per line -> docs/bom-audit.md, out/bom-mpn.csv
(manufacturer + MPN). Netlist connectivity unchanged, ERC 0, checkpins ok.

Co-Authored-By: Claude Opus 5.5 <noreply@anthropic.com>
Parts:
- C63: LCSC C23733 -> C1779
- C64: LCSC TBD-F5 -> C1622
- R83: LCSC TBD-F5 -> C17667
- R84: LCSC TBD-F5 -> C4310
- R85: LCSC TBD-F5 -> C17880
- R86: LCSC TBD-F5 -> C5713309
- R88: LCSC TBD-F5 -> C2933464
- R89: LCSC TBD-F5 -> C21841
Changed lines of the file:
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@@
 			)
 		)
-		(property "LCSC" "TBD-F5"
+		(property "LCSC" "C17667"
 			(at 248.92 96.52 0)
 			(hide yes)
@@
 			)
 		)
-		(property "LCSC" "TBD-F5"
+		(property "LCSC" "C4310"
 			(at 261.62 106.68 0)
 			(hide yes)
@@
 			)
 		)
-		(property "LCSC" "C23733"
+		(property "LCSC" "C1779"
 			(at 96.52 162.56 0)
 			(hide yes)
@@
 			)
 		)
-		(property "LCSC" "TBD-F5"
+		(property "LCSC" "C1622"
 			(at 152.4 162.56 0)
 			(hide yes)
@@
 			)
 		)
-		(property "LCSC" "TBD-F5"
+		(property "LCSC" "C17880"
 			(at 55.88 203.2 0)
 			(hide yes)
@@
 			)
 		)
-		(property "LCSC" "TBD-F5"
+		(property "LCSC" "C5713309"
 			(at 68.58 213.36 0)
 			(hide yes)
@@
 			)
 		)
-		(property "LCSC" "TBD-F5"
+		(property "LCSC" "C2933464"
 			(at 114.3 236.22 0)
 			(hide yes)
@@
 			)
 		)
-		(property "LCSC" "TBD-F5"
+		(property "LCSC" "C21841"
 			(at 127 246.38 0)
 			(hide yes)

Commit message: Pre-order verification review: 12 would-fail faults fixed, report added
Schematic (tools/sheets.py, sheets regenerated):
- D2 SMDJ100A: D_Zener symbol, cathode to VIN_P (was drawn forward with
  the bidirectional D_TVS symbol)
- D10/D11 BAV99 clamps: pin 1 (anode) GND, pin 2 (cathode) 3V3 (KiCad's
  hidden K/A/K pin names contradict the Nexperia pinout)
- D5/D6: BAV70 common-cathode replaces the mirrored BAV99 (opto LED was
  bypassed)
- U8 TXB0104 OE: 10k/100k = 1.64 V (47k/10k gave 0.32 V, UART disabled)
- R82 0.1R: EG11752 2 A peak limit (0R disabled it)
- D7/D8 flyback cathodes to VIN_P behind D1 (reverse-polarity path via
  the Q1/Q2 body diodes), VIN_P exported as a hierarchical net
- Q1/Q2 gate pulldown 100k (4.89 V; 10k gave 4.07 V), DI pull-up 220k,
  R91 51k USIM_DET pull-up, PESD5V0L5UY SIM ESD, X7R 1uF/4.7uF, 100k
  C149504, comments and notes corrected

Board (DRC-gated routes via tools/manual_routes.py + tools/board_fixes.py):
- D2/D10/D11 turned, NRST via moved, VIN trunk re-laid around D7/D8,
  VIN_P B.Cu run to D1, R91 on B.Cu, VBAT_BT 0.6 mm F.Cu to J2, SW_CHG
  0.4 mm, PMID 0.3/0.5 mm, DNP flags, C61<->C80 swap, 28 RF stitching
  vias, 9 vias under U5's pad; values updated
- manual_routes: delvia/padnet/rotate/value/move ops, ACCEPT_EQUAL

Checks: parity 0 mismatches (212 parts, 727 pad nets), ERC 0 errors,
pin checklist pass, DRC 0 errors / 0 unconnected, BOM audit 76/76 clean.

Docs: firmware-notes FW-6/8/13/14/17 + FW-18..22, BV-1/5/6/7; handoff and
installation sheet corrected (12 V floor, DI not isolated, values);
design-log entry; docs/verification-report.pdf (OK / NOT OK per item).

Co-Authored-By: Claude Fable 5.1 <noreply@anthropic.com>
Parts:
- C61, C68, C69, C75: LCSC C15849 -> C106858
- C63: LCSC C1779 -> C354262
- D2: symbol Device:D_TVS -> Device:D_Zener
- R81: LCSC C17407 -> C149504
- R82: value 0R (F-12) -> 0.1R; LCSC C17477 -> C327057
Connections:
- net GND: now also D2.2 (A); no longer D2.1 (A1)
- net VIN_P: now also D2.1 (K); no longer D2.2 (A2)
Other:
- note added: "Front end: F1 (250 VAC / 125 VDC, 100 A DC interrupt) -> D1 S3M reverse block -> D2 SMDJ100A 3kW -> R80 1R 2512 anti-surge (F-15 approved) -> buck. Margin at 3.7A clamp: 34.9%. R80 at the 10.5V floor, full load: V_B=9.16V, I=0.644A, 0.41W. 10R was a brown-out (no load-line solution) - see design-log F-15."
- note added: "U5 EG11752: EN 100k from VCC (per fig 6-2); VB-VS 100nF boot; IS via R82 0.1R -> 2 A peak limit (0.2 V / R_IS; BV-1 characterise); FB 4.3k/1.5k -> 5.03V; L 150uH (Isat 2.7A); SS3200 freewheel. #1 bench test: 100V in, 0.7-1A out, Ton~455ns."
- note removed: "Front end: F1 (250 VDC interrupt) -> D1 S3M reverse block -> D2 SMDJ100A 3kW -> R80 1R 2512 anti-surge (F-15 approved) -> buck. Margin at 3.7A clamp: 34.9%. R80 at the 10.5V floor, full load: V_B=9.16V, I=0.644A, 0.41W. 10R was a brown-out (no load-line solution) - see design-log F-15."
- note removed: "U5 EG11752: EN 100k from VCC (per fig 6-2); VB-VS 100nF boot; IS via R82 0R - F-12: no R_IS formula in the V1.0 datasheet, bench/FAE item; FB 4.3k/1.5k -> 5.03V; L 150uH (Isat 2.7A); SS3200 freewheel. #1 bench test: 100V in, 0.7-1A out, Ton~455ns."
Changed lines of the file:
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@@
 		)
 	)
-	(label "VIN_P"
+	(hierarchical_label "VIN_P"
+		(shape output)
 		(at 66.04 50.8 180)
 		(effects
@@
 				(size 1.27 1.27)
 			)
-			(justify right bottom)
+			(justify right)
 		)
 	)
 	(wire
 		(pts
-			(xy 97.79 63.5) (xy 101.6 63.5)
+			(xy 90.17 63.5) (xy 86.36 63.5)
 		)
 		(stroke
@@
 	)
 	(label "VIN_P"
-		(at 101.6 63.5 0)
+		(at 86.36 63.5 180)
 		(effects
 			(font
 				(size 1.27 1.27)
 			)
-			(justify left bottom)
+			(justify right bottom)
 		)
 	)
 	(wire
 		(pts
-			(xy 90.17 63.5) (xy 86.36 63.5)
+			(xy 97.79 63.5) (xy 101.6 63.5)
 		)
 		(stroke
@@
 		)
 	)
-	(text "Front end: F1 (250 VDC interrupt) -> D1 S3M reverse block -> D2 SMDJ100A 3kW -> R80 1R 2512 anti-surge (F-15 approved) -> buck. Margin at 3.7A clamp: 34.9%. R80 at the 10.5V floor, full load: V_B=9.16V, I=0.644A, 0.41W. 10R was a brown-out (no load-line solution) - see design-log F-15."
+	(text "Front end: F1 (250 VAC / 125 VDC, 100 A DC interrupt) -> D1 S3M reverse block -> D2 SMDJ100A 3kW -> R80 1R 2512 anti-surge (F-15 approved) -> buck. Margin at 3.7A clamp: 34.9%. R80 at the 10.5V floor, full load: V_B=9.16V, I=0.644A, 0.41W. 10R was a brown-out (no load-line solution) - see design-log F-15."
 		(exclude_from_sim no)
 		(at 38.1 35.56 0)
@@
 		)
 	)
-	(text "U5 EG11752: EN 100k from VCC (per fig 6-2); VB-VS 100nF boot; IS via R82 0R - F-12: no R_IS formula in the V1.0 datasheet, bench/FAE item; FB 4.3k/1.5k -> 5.03V; L 150uH (Isat 2.7A); SS3200 freewheel. #1 bench test: 100V in, 0.7-1A out, Ton~455ns."
+	(text "U5 EG11752: EN 100k from VCC (per fig 6-2); VB-VS 100nF boot; IS via R82 0.1R -> 2 A peak limit (0.2 V / R_IS; BV-1 characterise); FB 4.3k/1.5k -> 5.03V; L 150uH (Isat 2.7A); SS3200 freewheel. #1 bench test: 100V in, 0.7-1A out, Ton~455ns."
 		(exclude_from_sim no)
 		(at 190.5 121.92 0)
@@
 	)
 	(symbol
-		(lib_id "Device:D_TVS")
+		(lib_id "Device:D_Zener")
 		(at 93.98 63.5 0)
 		(unit 1)
@@
 	(symbol
 		(lib_id "power:GND")
-		(at 86.36 63.5 0)
+		(at 101.6 63.5 0)
 		(unit 1)
 		(exclude_from_sim no)
@@
 		(fields_autoplaced yes)
 		(property "Reference" "#PWR149"
-			(at 86.36 55.88 0)
+			(at 101.6 55.88 0)
 			(effects
 				(font
@@
 		)
 		(property "Value" "GND"
-			(at 86.36 63.5 0)
+			(at 101.6 63.5 0)
 			(hide yes)
 			(effects
@@
 			)
 		)
-		(property "LCSC" "C15849"
+		(property "LCSC" "C106858"
 			(at 254 35.56 0)
 			(hide yes)
@@
 			)
 		)
-		(property "LCSC" "C17407"
+		(property "LCSC" "C149504"
 			(at 241.3 35.56 0)
 			(hide yes)
@@
 			)
 		)
-		(property "Value" "0R (F-12)"
+		(property "Value" "0.1R"
 			(at 200.66 71.12 0)
 			(effects
@@
 			)
 		)
-		(property "LCSC" "C17477"
+		(property "LCSC" "C327057"
 			(at 200.66 76.2 0)
 			(hide yes)
@@
 			)
 		)
-		(property "LCSC" "C15849"
+		(property "LCSC" "C106858"
 			(at 71.12 162.56 0)
 			(hide yes)
@@
 			)
 		)
-		(property "LCSC" "C1779"
+		(property "LCSC" "C354262"
 			(at 96.52 162.56 0)
 			(hide yes)
@@
 			)
 		)
-		(property "LCSC" "C15849"
+		(property "LCSC" "C106858"
 			(at 261.62 205.74 0)
 			(hide yes)
@@
 			)
 		)
-		(property "LCSC" "C15849"
+		(property "LCSC" "C106858"
 			(at 299.72 205.74 0)
 			(hide yes)

Commit message: BOM: one LCSC part per line (C75 "1uF 25V" -> "1uF", C76 -> "100nF")
JLCPCB's assembly upload leaves a part unselected when the same part number
appears on two BOM lines - it cannot tell which line to buy for. C75 and C76
carried their voltage rating in the Value field, so they grouped separately
from the identical 1 uF and 100 nF parts. The rating belongs to the part, not
the label. Release now fails on a duplicate part number, as it does on a
BOM/CPL designator mismatch.

Package rebuilt: out/telematics-tracker-mfg-2026-09-30-91e36f5.zip

Co-Authored-By: Claude Opus 5 <noreply@anthropic.com>
Parts:
- C75: value 1uF 25V -> 1uF
- C76: value 100nF 25V -> 100nF
Changed lines of the file:
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@@
 			)
 		)
-		(property "Value" "1uF 25V"
+		(property "Value" "1uF"
 			(at 254 30.48 0)
 			(effects
@@
 			)
 		)
-		(property "Value" "100nF 25V"
+		(property "Value" "100nF"
 			(at 200.66 38.1 0)
 			(effects
